Commit message: changed urdf

File: models/solo12dof_quadruped/solo12dof_quadruped.urdf (robot description, URDF)
Before this commit: robot solo12dof_quadruped, 13 links, 12 joints
Links:
- link hip_fe_rl: geometry visual mesh filename=meshes/solo12_hip_fe_hl.stl
Joints:
- joint hip_fe_fl: limit lower=-2.44 upper=2.44 effort=18 velocity=40 -> lower=-1.3089969389957472 upper=2.443460952792061 effort=18 velocity=40
- joint hip_fe_fr: limit lower=-2.44 upper=2.44 effort=18 velocity=40 -> lower=-2.443460952792061 upper=1.3089969389957472 effort=18 velocity=40
- joint hip_fe_rl: limit lower=-2.44 upper=2.44 effort=18 velocity=40 -> lower=-1.3089969389957472 upper=2.443460952792061 effort=18 velocity=40
- joint hip_fe_rr: limit lower=-2.44 upper=2.44 effort=18 velocity=40 -> lower=-2.443460952792061 upper=1.3089969389957472 effort=18 velocity=40

Commit message: changed urdf

File: models/solo12dof_quadruped/solo12dof_quadruped.urdf (robot description, URDF)
Before this commit: robot solo12dof_quadruped, 13 links, 12 joints
Links:
- link LLM_fl: geometry visual mesh filename=meshes/solo12_lower_leg_v2_left_side.STL
- link LLM_fr: geometry visual mesh filename=meshes/solo12_lower_leg_v2_right_side.obj
- link LLM_rl: geometry visual mesh filename=meshes/solo12_lower_leg_v2_left_side.STL
- link LLM_rr: geometry collision mesh filename=package://solo12dof_quadruped/meshes/solo12_lower_leg_v2_ri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; visual mesh filename=meshes/solo12_lower_leg_v2_right_side.STL
- link ULM_fl: geometry visual mesh filename=meshes/solo12_upper_leg_left_side.stl
- link ULM_fr: geometry collision mesh filename=package://solo12dof_quadruped/meshes/solo12_upper_leg_right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; visual mesh filename=meshes/solo12_upper_leg_right_side.stl
- link ULM_rl: geometry visual mesh filename=meshes/solo12_upper_leg_left_side.stl
- link ULM_rr: geometry visual mesh filename=meshes/solo12_upper_leg_right_side.stl
Joints:
- joint LLM_fl: limit lower=-3.141592653589793 upper=3.141592653589793 effort=0 velocity=0 -> lower=-3.141592653589793 upper=3.141592653589793 effort=18 velocity=40
- joint LLM_fr: limit lower=-3.141592653589793 upper=3.141592653589793 effort=0 velocity=0 -> lower=-3.141592653589793 upper=3.141592653589793 effort=18 velocity=40
- joint LLM_rl: limit lower=-3.141592653589793 upper=3.141592653589793 effort=0 velocity=0 -> lower=-3.141592653589793 upper=3.141592653589793 effort=18 velocity=40
- joint LLM_rr: limit lower=-3.141592653589793 upper=3.141592653589793 effort=0 velocity=0 -> lower=-3.141592653589793 upper=3.141592653589793 effort=18 velocity=40
- joint ULM_fl: limit lower=-1.5707963267948966 upper=1.5707963267948966 effort=0 velocity=0 -> lower=-1.5707963267948966 upper=1.5707963267948966 effort=18 velocity=40
- joint ULM_fr: limit lower=-1.5707963267948966 upper=1.5707963267948966 effort=0 velocity=0 -> lower=-1.5707963267948966 upper=1.5707963267948966 effort=18 velocity=40
- joint ULM_rl: limit lower=-1.5707963267948966 upper=1.5707963267948966 effort=0 velocity=0 -> lower=-1.5707963267948966 upper=1.5707963267948966 effort=18 velocity=40
- joint ULM_rr: limit lower=-1.5707963267948966 upper=1.5707963267948966 effort=0 velocity=0 -> lower=-1.5707963267948966 upper=1.5707963267948966 effort=18 velocity=40

Commit message: changed urdf

File: models/solo12dof_quadruped/solo12dof_quadruped.urdf (robot description, URDF)
Before this commit: robot solo12dof_quadruped, 13 links, 12 joints
Links:
- link LLM_fl: geometry visual mesh filename=meshes/solo12_lower_leg_v2_left_side.obj
- link LLM_rl: geometry visual mesh filename=meshes/solo12_lower_leg_v2_left_side.obj
- link LLM_rr: geometry collision mesh filename=meshes/solo12_lower_leg_v2_right_side.obj; visual mesh filename=meshes/solo12_lower_leg_v2_right_side.obj
- link ULM_fl: geometry visual mesh filename=meshes/solo12_upper_leg_left_side.obj
- link ULM_fr: geometry collision mesh filename=meshes/solo12_upper_leg_right_side.obj; visual mesh filename=meshes/solo12_upper_leg_right_side.obj
- link ULM_rl: geometry visual mesh filename=meshes/solo12_upper_leg_left_side.obj
- link ULM_rr: geometry visual mesh filename=meshes/solo12_upper_leg_right_side.obj
- link hip_fe_fl: geometry visual mesh filename=meshes/solo12_hip_fe_fl.obj
- link hip_fe_fr: geometry visual mesh filename=meshes/solo12_hip_fe_fr.obj
- link hip_fe_rl: geometry visual mesh filename=meshes/solo12_hip_fe_hl.obj
- link hip_fe_rr: geometry collision mesh filename=meshes/solo12_hip_fe_hr.obj; visual mesh filename=meshes/solo12_hip_fe_hr.obj

Commit message: try run robot, but problem maybe with bad converted meshes from .wtl to .obj

File: models/solo12dof_quadruped/solo12dof_quadruped.urdf (robot description, URDF)
Before this commit: robot solo12dof_quadruped, 13 links, 12 joints
Links:
- removed link base_link
- added link LF_FOOT; collision sphere radius=0.0159; visual sphere radius=0.0159
- added link LH_FOOT; collision sphere radius=0.0159; visual sphere radius=0.0159
- added link RF_FOOT; collision sphere radius=0.0159; visual sphere radius=0.0159
- added link RH_FOOT; collision sphere radius=0.0159; visual sphere radius=0.0159
- added link body, mass 1258.31807296e-3; visual mesh filename=meshes/solo12_base.obj
Joints:
- added joint foot_fl: type fixed, parent LLM_fl, child LF_FOOT, origin xyz=0.0 0.0 0.0 rpy=0.0 0.0 0.0
- added joint foot_fr: type fixed, parent LLM_fr, child RF_FOOT, origin xyz=0.0 0.0 0.0 rpy=0.0 0.0 0.0
- added joint foot_rl: type fixed, parent LLM_rl, child LH_FOOT, origin xyz=0.0 0.0 0.0 rpy=0.0 0.0 0.0
- added joint foot_rr: type fixed, parent LLM_rr, child RH_FOOT, origin xyz=0.0 0.0 0.0 rpy=0.0 0.0 0.0
- joint hip_fe_fl: parent base_link -> body
- joint hip_fe_fr: parent base_link -> body
- joint hip_fe_rl: parent base_link -> body
- joint hip_fe_rr: parent base_link -> body
