Commit message: solo12_base.obj and solo_12_base.STL tested and they doesn't work

File: models/mini_cheetah/mini_cheetah_mesh.urdf (robot description, URDF)
Before this commit: robot mini_cheetah, 17 links, 16 joints
Links:
- link body: geometry visual mesh filename=meshes/mini_body.obj

Commit message: added correct base mesh and chenged it's color

File: models/mini_cheetah/mini_cheetah_mesh.urdf (robot description, URDF)
Before this commit: robot mini_cheetah, 17 links, 16 joints
Links:
- link body: geometry visual mesh filename=meshes/solo_12_base.obj

Commit message: body mass reduced to 2.5 kg

File: models/mini_cheetah/mini_cheetah_mesh.urdf (robot description, URDF)
Before this commit: robot mini_cheetah, 17 links, 16 joints
Links:
- link body: mass 3.3 -> 2.5

Commit message: added .mtl for body, front left leg from solo12, but position being clarified

File: models/mini_cheetah/mini_cheetah_mesh.urdf (robot description, URDF)
Before this commit: robot mini_cheetah, 17 links, 16 joints
Links:
- link abduct_fl: geometry visual mesh filename=meshes/solo12_hip_fe_fl.obj
- link shank_fl: geometry visual mesh filename=meshes/solo12_lower_leg_v2_left_side.obj
- link thigh_fl: geometry visual mesh filename=meshes/solo12_upper_leg_left_side.obj
Joints:
- joint torso_to_abduct_fl_j: origin xyz=0.19 0.049 0.0 rpy=0 0 0 -> xyz=0.19 0.049 0.0  rpy=0 0 0

Commit message: mass of body returned back, coordinates of joints of hip aa modules setup as solo12 robot, dt decrease to 1e-3

File: models/mini_cheetah/mini_cheetah_mesh.urdf (robot description, URDF)
Before this commit: robot mini_cheetah, 17 links, 16 joints
Links:
- link LF_FOOT: mass None -> 0.005
- link LH_FOOT: mass None -> 0.005
- link RF_FOOT: mass None -> 0.005
- link RH_FOOT: mass None -> 0.005
- link body: mass 2.5 -> 3.3
Joints:
- joint torso_to_abduct_fl_j: origin xyz=0.19 0.049 0.0  rpy=0 0 0 -> xyz=0.2141 0.0875 0.0  rpy=0 0 0
- joint torso_to_abduct_fr_j: origin xyz=0.19 -0.049 0.0 rpy=0 0 0 -> xyz=0.2141 -0.0875 0.0 rpy=0 0 0
- joint torso_to_abduct_hl_j: origin xyz=-0.19 0.049 0.0 rpy=0 0 0 -> xyz=-0.2141 0.0875 0.0 rpy=0 0 0
- joint torso_to_abduct_hr_j: origin xyz=-0.19 -0.049 0.0 rpy=0 0 0 -> xyz=-0.2141 -0.0875 0.0 rpy=0 0 0

Commit message: changed joint position for all hip fe modules and work succesfully with ID method

File: models/mini_cheetah/mini_cheetah_mesh.urdf (robot description, URDF)
Before this commit: robot mini_cheetah, 17 links, 16 joints
Links:
- link abduct_fr: geometry visual mesh filename=meshes/solo12_hip_fe_fr.obj
- link abduct_hl: geometry visual mesh filename=meshes/solo12_hip_fe_hl.obj
- link abduct_hr: geometry visual mesh filename=meshes/solo12_hip_fe_hr.obj

Commit message: all legs meshes added, position of jionts of ULM modules setup and check verified

File: models/mini_cheetah/mini_cheetah_mesh.urdf (robot description, URDF)
Before this commit: robot mini_cheetah, 17 links, 16 joints
Links:
- link shank_fr: geometry visual mesh filename=meshes/solo12_lower_leg_v2_right_side.obj
- link shank_hl: geometry visual mesh filename=meshes/solo12_lower_leg_v2_left_side.obj
- link shank_hr: geometry visual mesh filename=meshes/solo12_lower_leg_v2_right_side.obj
- link thigh_fr: geometry visual mesh filename=meshes/solo12_upper_leg_right_side.obj
- link thigh_hl: geometry visual mesh filename=meshes/solo12_upper_leg_left_side.obj
- link thigh_hr: geometry visual mesh filename=meshes/solo12_upper_leg_right_side.obj
Joints:
- joint abduct_fl_to_thigh_fl_j: origin xyz=0.0 0.062 0.00 rpy=0.0 0.0 0.0 -> xyz=-19.65e-3 14e-3 0 rpy=0.0 0.0 0.0
- joint abduct_fr_to_thigh_fr_j: origin xyz=0.0 -0.062 0.00 rpy=0.0 0.0 0.0 -> xyz=-19.65e-3 -14e-3 0 rpy=0.0 0.0 0.0
- joint abduct_hl_to_thigh_hl_j: origin xyz=0.0 0.062 0.00 rpy=0.0 0.0 0.0 -> xyz=19.65e-3 14e-3 0  rpy=0.0 0.0 0.0
- joint abduct_hr_to_thigh_hr_j: origin xyz=0.0 -0.062 0.00 rpy=0.0 0.0 0.0 -> xyz=19.65e-3 -14e-3 0 rpy=0.0 0.0 0.0

Commit message: changed contact's spheres radiuses

File: models/mini_cheetah/mini_cheetah_mesh.urdf (robot description, URDF)
Before this commit: robot mini_cheetah, 17 links, 16 joints
Links:
- link LF_FOOT: geometry collision sphere radius=0.0159; visual sphere radius=0.0159
- link LH_FOOT: geometry collision sphere radius=0.0159; visual sphere radius=0.0159
- link RF_FOOT: geometry collision sphere radius=0.0159; visual sphere radius=0.0159
- link RH_FOOT: geometry collision sphere radius=0.0159; visual sphere radius=0.0159

Commit message: all masses match with the solo12 robot

File: models/mini_cheetah/mini_cheetah_mesh.urdf (robot description, URDF)
Before this commit: robot mini_cheetah, 17 links, 16 joints
Links:
- link abduct_fl: mass 0.54 -> 143.68024490e-3
- link abduct_fr: mass 0.54 -> 143.68024490e-3
- link abduct_hl: mass 0.54 -> 143.68024490e-3
- link abduct_hr: mass 0.54 -> 143.68024490e-3
- link body: mass 3.3 -> 1258.31807296e-3
- link shank_fl: mass 0.064 -> 44.08831168e-3
- link shank_fr: mass 0.064 -> 44.08831168e-3
- link shank_hl: mass 0.064 -> 44.08831168e-3
- link shank_hr: mass 0.064 -> 44.08831168e-3
- link thigh_fl: mass 0.634 -> 144.14222037e-3
- link thigh_fr: mass 0.634 -> 144.14222037e-3
- link thigh_hl: mass 0.634 -> 144.14222037e-3
- link thigh_hr: mass 0.634 -> 144.14222037e-3

Commit message: all LLM modules joint's x y match with solo12 robot

File: models/mini_cheetah/mini_cheetah_mesh.urdf (robot description, URDF)
Before this commit: robot mini_cheetah, 17 links, 16 joints
Joints:
- joint thigh_fl_to_knee_fl_j: origin xyz=0.0 0.0 -0.209 rpy=0.0 0 0.0 -> xyz=0.0 37e-3 -0.209 rpy=0.0 0 0.0
- joint thigh_fr_to_knee_fr_j: origin xyz=0.0 0.0 -0.209 rpy=0.0 0 0.0 -> xyz=0.0 -37e-3 -0.209 rpy=0.0 0 0.0
- joint thigh_hl_to_knee_hl_j: origin xyz=0.0 0.0 -0.209 rpy=0.0 0 0.0 -> xyz=0.0 37e-3 -0.209 rpy=0.0 0 0.0
- joint thigh_hr_to_knee_hr_j: origin xyz=0.0 0.0 -0.209 rpy=0.0 0 0.0 -> xyz=0.0 -37e-3 -0.209 rpy=0.0 0 0.0

Commit message: foot coord clarify

File: models/mini_cheetah/mini_cheetah_mesh.urdf (robot description, URDF)
Before this commit: robot mini_cheetah, 17 links, 16 joints
Links:
- link LF_FOOT: geometry collision sphere radius=0.0162; visual sphere radius=0.0162
- link LH_FOOT: geometry collision sphere radius=0.0162; visual sphere radius=0.0162
- link RF_FOOT: geometry collision sphere radius=0.0162; visual sphere radius=0.0162
- link RH_FOOT: geometry collision sphere radius=0.0162; visual sphere radius=0.0162
Joints:
- joint abduct_hr_to_thigh_hr_j: origin xyz=19.65e-3 -14e-3 0 rpy=0.0 0.0 0.0 -> xyz=19.65e-3 -14e-3 0 rpy=0.0 0 0
- joint shank_fl_to_foot_fl: origin xyz=0.0 0.0 -0.190 rpy=0.0 0.0 0.0 -> xyz=0.0 15.5e-3 -0.190 rpy=0.0 0.0 0.0
- joint shank_fr_to_foot_fr: origin xyz=0.0 0.0 -0.190 rpy=0.0 0.0 0.0 -> xyz=0.0 -15.5e-3 -0.190 rpy=0.0 0.0 0.0
- joint shank_hl_to_foot_hl: origin xyz=0.0 0.0 -0.190 rpy=0.0 0.0 0.0 -> xyz=0.0 15.5e-3 -0.190 rpy=0.0 0.0 0.0
- joint shank_hr_to_foot_hr: origin xyz=0.0 0.0 -0.190 rpy=0.0 0.0 0.0 -> xyz=0.0 -15.5e-3 -0.190 rpy=0.0 0.0 0.0
- joint thigh_hr_to_knee_hr_j: origin xyz=0.0 -37e-3 -0.209 rpy=0.0 0 0.0 -> xyz=0.0 -37e-3 -0.209 rpy=0.0 0 0

Commit message: all parameters match with solo12 robotm, but somehow the same error

File: models/mini_cheetah/mini_cheetah_mesh.urdf (robot description, URDF)
Before this commit: robot mini_cheetah, 17 links, 16 joints
Links:
- link LF_FOOT: geometry collision sphere radius=0.018; visual sphere radius=0.018
- link LH_FOOT: geometry collision sphere radius=0.018; visual sphere radius=0.018
- link RF_FOOT: geometry collision sphere radius=0.018; visual sphere radius=0.018
- link RH_FOOT: geometry collision sphere radius=0.018; visual sphere radius=0.018
Joints:
- joint shank_fl_to_foot_fl: origin xyz=0.0 15.5e-3 -0.190 rpy=0.0 0.0 0.0 -> xyz=0.0 7.5e-3 -0.16 rpy=0.0 0.0 0.0
- joint shank_fr_to_foot_fr: origin xyz=0.0 -15.5e-3 -0.190 rpy=0.0 0.0 0.0 -> xyz=0.0 -7.5e-3 -0.16 rpy=0.0 0.0 0.0
- joint shank_hl_to_foot_hl: origin xyz=0.0 15.5e-3 -0.190 rpy=0.0 0.0 0.0 -> xyz=0.0 7.5e-3 -0.16 rpy=0.0 0.0 0.0
- joint shank_hr_to_foot_hr: origin xyz=0.0 -15.5e-3 -0.190 rpy=0.0 0.0 0.0 -> xyz=0.0 -7.5e-3 -0.16 rpy=0.0 0.0 0.0
- joint thigh_fl_to_knee_fl_j: origin xyz=0.0 37e-3 -0.209 rpy=0.0 0 0.0 -> xyz=0.0 37e-3 -0.16 rpy=0.0 0 0.0
- joint thigh_fr_to_knee_fr_j: origin xyz=0.0 -37e-3 -0.209 rpy=0.0 0 0.0 -> xyz=0.0 -37e-3 -0.16 rpy=0.0 0 0.0
- joint thigh_hl_to_knee_hl_j: origin xyz=0.0 37e-3 -0.209 rpy=0.0 0 0.0 -> xyz=0.0 37e-3 -0.16 rpy=0.0 0 0.0
- joint thigh_hr_to_knee_hr_j: origin xyz=0.0 -37e-3 -0.209 rpy=0.0 0 0 -> xyz=0.0 -37e-3 -0.16 rpy=0.0 0 0

Commit message: I solved the problem by adding 92 line of code p_body_nom[2] = 0.24094614699109293 to clf_controller.py. I think this way you can make any controller work.

File: models/mini_cheetah/mini_cheetah_mesh.urdf (robot description, URDF)
Before this commit: robot mini_cheetah, 17 links, 16 joints
Links:
- link LF_FOOT: geometry collision sphere radius=0.018
- link LH_FOOT: geometry collision sphere radius=0.018
- link RF_FOOT: geometry collision sphere radius=0.018
- link RH_FOOT: geometry collision sphere radius=0.018

Commit message: new branch for version with two parts of one lower leg module imitating flexible leg

File: models/mini_cheetah/mini_cheetah_mesh.urdf (robot description, URDF)
Before this commit: robot mini_cheetah, 17 links, 16 joints
Links:
- added link lower_leg_L_fl, mass 44.08831168e-3; visual mesh filename=meshes/solo12_lower_leg_v2_left_side.obj
- link shank_fl: mass 44.08831168e-3 -> 23.48772094e-3; geometry visual mesh filename=meshes/solo12_lower_leg_H.obj
Joints:
- added joint lower_leg_joint_fl: type continuous, parent thigh_fl, child shank_fl, origin xyz=0.0 37e-3 -0.16 rpy=0.0 0 0.0, axis 0 -1 0, limit lower=-2.6 upper=2.6 effort=26 velocity=26

Commit message: in the URDF added new joints and links with correct parameters, contact point coordinates approptiatly changed, trash collision deleted, obj files corrected according with old MTL file

File: models/mini_cheetah/mini_cheetah_mesh.urdf (robot description, URDF)
Before this commit: robot mini_cheetah, 18 links, 17 joints
Links:
- link lower_leg_L_fl: mass 44.08831168e-3 -> 14.20602001e-3; geometry visual mesh filename=meshes/solo12_lower_leg_L.obj
Joints:
- joint lower_leg_joint_fl: child shank_fl -> lower_leg_L_fl; origin xyz=0.0 37e-3 -0.16 rpy=0.0 0 0.0 -> xyz=0.0 7.5e-3 -0.08 rpy=0.0 0 0.0; parent thigh_fl -> shank_fl
- joint shank_fl_to_foot_fl: origin xyz=0.0 7.5e-3 -0.16 rpy=0.0 0.0 0.0 -> xyz=0.0 0 -0.08 rpy=0.0 0.0 0.0

Commit message: in URDF corrected child link reference in shank_fl_foot_fl joint and delete colision

File: models/mini_cheetah/mini_cheetah_mesh.urdf (robot description, URDF)
Before this commit: robot mini_cheetah, 18 links, 17 joints
Joints:
- joint shank_fl_to_foot_fl: parent shank_fl -> lower_leg_L_fl

Commit message: add torsion spring instance to URDF

File: models/mini_cheetah/mini_cheetah_mesh.urdf (robot description, URDF)
Before this commit: robot mini_cheetah, 18 links, 17 joints
Joints:
- joint lower_leg_joint_fl: limit lower=-2.6 upper=2.6 effort=26 velocity=26 -> (none)

Commit message: new joint's type cheged on fixed, I have an idea to implement nonlinear flexible link between 2 joints in lower leg's part: like nonlinear spring or with drake's FEM

File: models/mini_cheetah/mini_cheetah_mesh.urdf (robot description, URDF)
Before this commit: robot mini_cheetah, 18 links, 17 joints
Links:
- link LF_FOOT: geometry collision sphere radius=0.018; visual sphere radius=0.018
- link lower_leg_L_fl: geometry visual mesh filename=meshes/solo12_lower_leg_L.obj scale=0.001 0.001 0.001
- link shank_fl: geometry visual mesh filename=meshes/solo12_lower_leg_H.obj scale=0.001 0.001 0.001
Joints:
- joint lower_leg_joint_fl: limit (none) -> lower=-2.6 upper=2.6 effort=18 velocity=40; type continuous -> fixed

Commit message: meshes was updated with correct sizes and origins, now leg represent 2 links with 1 joint

File: models/mini_cheetah/mini_cheetah_mesh.urdf (robot description, URDF)
Before this commit: robot mini_cheetah, 18 links, 17 joints
Links:
- link lower_leg_L_fl: geometry visual mesh filename=meshes/solo12_lower_leg_L.obj scale=1 1 1
- link shank_fl: geometry visual mesh filename=meshes/solo12_lower_leg_H.obj scale=1 1 1

Commit message: one leg is divided on 3 links with 2 fixed joints, in the next we will change center link on flexible one. But I concerned with the robot length of step, it is very long, so the robot could fall after center link getting flexible.

File: models/mini_cheetah/mini_cheetah_mesh.urdf (robot description, URDF)
Before this commit: robot mini_cheetah, 18 links, 17 joints
Links:
- added link lower_leg_center_fl, mass 1e-3; visual box size=10e-3 10e-3 14e-3
- link LH_FOOT: geometry collision sphere radius=0.018; visual sphere radius=0.018
- link RF_FOOT: geometry collision sphere radius=0.018; visual sphere radius=0.018
- link RH_FOOT: geometry collision sphere radius=0.018; visual sphere radius=0.018
Joints:
- removed joint lower_leg_joint_fl
- added joint lower_leg_joint1_fl: type fixed, parent shank_fl, child lower_leg_center_fl, origin xyz=0.0 7.95e-3 -0.0725 rpy=0.0 0 0.0, axis 0 -1 0
- added joint lower_leg_joint2_fl: type fixed, parent lower_leg_center_fl, child lower_leg_L_fl, origin xyz=0.0 0 -0.014 rpy=0.0 0 0.0, axis 0 -1 0
- joint shank_fr_to_foot_fr: origin xyz=0.0 -7.5e-3 -0.16 rpy=0.0 0.0 0.0 -> xyz=0.0 -7.95e-3 -0.16 rpy=0.0 0.0 0.0
- joint shank_hl_to_foot_hl: origin xyz=0.0 7.5e-3 -0.16 rpy=0.0 0.0 0.0 -> xyz=0.0 7.95e-3 -0.16 rpy=0.0 0.0 0.0
- joint shank_hr_to_foot_hr: origin xyz=0.0 -7.5e-3 -0.16 rpy=0.0 0.0 0.0 -> xyz=0.0 -7.95e-3 -0.16 rpy=0.0 0.0 0.0

Commit message: new deformable example

File: models/mini_cheetah/mini_cheetah_mesh.urdf (robot description, URDF)
Before this commit: robot mini_cheetah, 19 links, 18 joints
Joints:
- joint lower_leg_joint1_fl: origin xyz=0.0 7.95e-3 -0.0725 rpy=0.0 0 0.0 -> xyz=0.0 7.95e-3 -0.073 rpy=0.0 0 0.0
- joint shank_fl_to_foot_fl: origin xyz=0.0 0 -0.08 rpy=0.0 0.0 0.0 -> xyz=0.0 0 -0.073 rpy=0.0 0.0 0.0
